Commit message: minor fixes

File: depthai_descriptions/urdf/include/base_macro.urdf.xacro (robot description, xacro)
@@ -44,6 +44,6 @@
             <xacro:property name="imu_offset_y" value="-0.037945" />
             <xacro:property name="imu_offset_z" value="-0.00079" />
-            <xacro:property name="imu_r" value="${M_PI}" />
-            <xacro:property name="imu_p" value="${M_PI/2.0}" />
+            <xacro:property name="imu_r" value="0" />
+            <xacro:property name="imu_p" value="-${M_PI/2.0}" />
             <xacro:property name="imu_y" value="0.0" />
         </xacro:if>
